Commit message: updated urdf with joint 2,4=-90 degrees

File: urdf/mycobot_pro_600.urdf (robot description, URDF)
Before this commit: robot firefighter, 7 links, 6 joints
Joints:
- joint joint3_to_joint2: origin xyz=0 0  0 rpy=1.5708 -1.5708 0 -> xyz=0 0  0 rpy=1.5708 0 0
- joint joint5_to_joint4: origin xyz=0.25 0  -0.1091 rpy=0 0 1.5708 -> xyz=0.25 0  -0.1091 rpy=0 0 0

Commit message: Updated files for ik

File: urdf/mycobot_pro_600.urdf (robot description, URDF)
Before this commit: robot firefighter, 7 links, 6 joints
Links:
- added link tool0; visual box size=0.01 0.01 0.01
Joints:
- added joint tool0_fixed: type fixed, parent link6, child tool0, origin xyz=0 0 0 rpy=0 0 0
